File: schematics/schematics.sch (KiCad schematic (older format))
At the start: 42 parts, among them J1-220V Screw_Terminal_01x02, J2 Screw_Terminal_01x02, J3 Screw_Terminal_01x02, J4 Screw_Terminal_01x02, J5 Screw_Terminal_01x02, SW1 SW_Push, SW2 SW_Push, SW3 SW_Push, SW4 SW_Push

Commit message: Finalize circuit for the LED strip
Parts:
- added D1: LED_BARG, symbol Device:LED_BARG
- added R10, R11, R9: R, symbol Device:R
- added T1, T2, T3: Q_NPN_BCE, symbol Device:Q_NPN_BCE
Connections:
- wire segments 138 -> 174
Other:
- moved on the sheet: SW1, SW2, SW3, SW4

Commit message: Make circuit look better
Parts:
- removed D4: DIODE, symbol pspice:DIODE
- removed D?: DS4, symbol pspice:DIODE
- removed JP?: Jumper, symbol Device:Jumper
- removed Q?: 2N2219, Package_TO_SOT_THT:TO-39-3, symbol Transistor_BJT:2N2219
- removed R7, R8: R, symbol Device:R
- removed U?: TLP185, Package_SO:SOIC-4_4.55x3.7mm_P2.54mm, symbol Isolator:TLP185
- added D?: DIODE, symbol pspice:DIODE
- added D?: DS3, symbol pspice:DIODE
- added JP? (x6): Jumper, symbol Device:Jumper
- added Q?: 2N2219, Package_TO_SOT_THT:TO-39-3, symbol Transistor_BJT:2N2219
- added R? (x2): R, symbol Device:R
- added U?: TLP185, Package_SO:SOIC-4_4.55x3.7mm_P2.54mm, symbol Isolator:TLP185
- renumbered J1-220V to J0-220V, J2 to J1, J3 to J2, J4 to J3, J5 to J4
Connections:
- net GNDREF: now also Q?.1 (E)
- net VCC: now also JP?.1, R?.1
- net at K?.6: now also D?.2 (A), JP?.2, U?.6
- net at K?.7, K?.8: now also JP?.2; no longer J3.2 (Pin_2)
- net at K?.7, K?.8: now also JP?.2; no longer J2.2 (Pin_2)
- net at K?.7, K?.8: now also JP?.2; no longer J1.2 (Pin_2)
- net at K?.2: now also D?.1 (K), Q?.3 (C)
- net at A?.22 (D7): now also SW4.1
- net at A?.23 (D8): now also SW3.1
- net at A?.24 (D9): now also SW2.1
- net at A?.25 (D10): now also SW1.1
- net at A?.7 (GND), T1.3 (E), T3.3 (E): now also JP?.2; no longer T2.3 (E)
- net at D1.3 (RK): now also JP?.2; no longer T3.2 (C)
- new net: J3.2 (Pin_2), JP?.1
- new net: J2.2 (Pin_2), JP?.1
- new net: J1.2 (Pin_2), JP?.1
- new net: JP?.1, T2.3 (E)
- new net: JP?.1, T3.2 (C)
- new net: Q?.2 (B), R?.1
- new net: R?.2, U?.1
- new net: D?.1 (K), U?.3
- new net: R?.2, U?.4
- now unconnected: A?.6 (GND)
Other:
- moved on the sheet: D1, R10, R11, R9, SW1, SW2, SW3, SW4, T1, T2, T3
